File: BulkyMIDI-32 Module/BulkyMIDI-32 Module.kicad_sch (KiCad schematic)
At the start: 63 parts, among them IC1 OLED, J1 DC IN, J10 AudioJack3, J2 MIDI OUT, J3 MIDI IN, J4 Faceplate, J5 MIDI THRU, J6 Serial, J7 Conn_Extras, J8 Module_Panel, J9 USB_C_Receptacle_USB2.0, M1 Mounting, M2 Mounting, M3 Mounting, M4 Mounting, SW1 SYNTH, SW2 ROM, SW3 VOL_DOWN, SW4 VOL_UP, U1 74HCT14, U2 H11L1M, U3 PCM5102A, U4 AMS1117-3.3, U5 AMS1117-3.3

Commit message: Compact and integrated DAC with both MT32Pi and Dexed support
Parts:
- removed J10: AudioJack3, symbol Connector_Audio:AudioJack3
- added C16, C17: 2n2, Capacitor_SMD:C_0402_1005Metric, symbol Device:C
- added C18, C24, C25: 100u, Capacitor_Tantalum_SMD:CP_EIA-3528-21_Kemet-B, symbol BulkyMIDI-32 Module-rescue:CP1-Device
- added C19, C23: 10u, Capacitor_SMD:C_0402_1005Metric, symbol Device:C
- added C20, C21, C22: 100n, Capacitor_SMD:C_0402_1005Metric, symbol Device:C
- added C26, C27, C28: 100uF, Capacitor_Tantalum_SMD:CP_EIA-3528-21_Kemet-B, symbol BulkyMIDI-32 Module-rescue:CP1-Device
- added J11: AudioJack4, Connector_Audio:Jack_3.5mm_PJ320D_Horizontal, symbol Connector_Audio:AudioJack4
- added JP7, JP8: P1_GND, Jumper:SolderJumper-3_P1.3mm_Open_RoundedPad1.0x1.5mm, symbol BulkyMIDI-32 Module-rescue:PowerSelect-I2C_OLED
- C1, C10, C11, C12, C13, C14, C15, C2, C3, C4, C7, C8, C9: footprint Capacitor_SMD:C_0805_2012Metric -> Capacitor_SMD:C_0402_1005Metric
- C5: footprint Capacitor_THT:CP_Radial_D6.3mm_P2.50mm -> Capacitor_Tantalum_SMD:CP_EIA-3528-21_Kemet-B
- C6: value 470uF -> 100u; footprint Capacitor_THT:CP_Radial_D8.0mm_P3.50mm -> Capacitor_Tantalum_SMD:CP_EIA-3528-21_Kemet-B
- R10, R11, R12, R13, R8, R9: footprint Resistor_SMD:R_0603_1608Metric -> Resistor_SMD:R_0402_1005Metric
Connections:
- net +3.3VA: now also C19.1, C20.1
- net +3.3VP: now also C22.1, C23.1
- net +3V3: now also JP8.1 (A); no longer J8.12 (VCC)
- net +5V: now also C10.1, C11.1, C14.1, U4.3 (VI), U5.3 (VI), C18.1, C21.1, C24.1, C25.1, C26.1, C27.1, C28.1
- net AUDIO_L: now also C17.1, J11.T
- net AUDIO_R: now also C16.1, J11.R1
- net GND: now also C16.2, C17.2, C18.2, C19.2, C20.2, C21.2, C22.2, C23.2, C24.2, C25.2, C26.2, C27.2, C28.2, J11.S, JP7.1 (A); no longer J8.11 (GND)
- net SW_DOWN_DEXED: now reaches A1.18 (GPIO24)
- net ENC_CLK_DEXED: now reaches A1.19 (MOSI0/GPIO10)
- net ENC_CLK_DEXED: now also JP8.3 (B)
- net ENC_DAT_DEXED: now reaches A1.21 (MISO0/GPIO9)
- net ENC_DAT_DEXED: now also JP7.3 (B)
- net ENC_SW_DEXED: now reaches A1.23 (SCLK0/GPIO11)
- new net: J8.11 (GND), JP7.2 (C)
- new net: J8.12 (VCC), JP8.2 (C)
- no-connect marks 32 -> 28
